File: bikesenseCap.sch (KiCad schematic (older format))
At the start: 43 parts

Commit message: Routing updated
Parts:
- removed D? (x4): LED_Small, symbol Device:LED_Small
- removed J? (x4): PAD, symbol cap1188:PAD
- removed R? (x4): 470, symbol Device:R_Small
- added D11: West, LEDs:LED_0805_HandSoldering, symbol Device:LED_Small
- added D12: NorthWest, LEDs:LED_0805_HandSoldering, symbol Device:LED_Small
- added D13: SouthWest, LEDs:LED_0805_HandSoldering, symbol Device:LED_Small
- added D14: North, LEDs:LED_0805_HandSoldering, symbol Device:LED_Small
- added D15: South, LEDs:LED_0805_HandSoldering, symbol Device:LED_Small
- added D16: NorthEast, LEDs:LED_0805_HandSoldering, symbol Device:LED_Small
- added D17: SouthEast, LEDs:LED_0805_HandSoldering, symbol Device:LED_Small
- added D18: East, LEDs:LED_0805_HandSoldering, symbol Device:LED_Small
- added R19, R21, R22, R27, R28, R31, R32, R35: 66, Resistors_SMD:R_0603_HandSoldering, symbol Device:R_Small
- added R20, R24, R25, R29, R30, R33, R34, R36: 100k, Resistors_SMD:R_0603_HandSoldering, symbol Device:R_Small
- added R23, R26: 10K, Resistors_SMD:R_0603_HandSoldering, symbol Device:R_Small
- added U3: TCA9534, digikey-footprints:SOIC-16_W7.5mm, symbol Interface_Expansion:TCA9534
- D1, D2: renamed from D?; footprint Diode_THT:D_DO-35_SOD27_P7.62mm_Horizontal -> Diodes_SMD:D_SOD-123
- D3, D4, D5, D6: renamed from D?; footprint (none) -> LEDs:LED_0603_HandSoldering
- J1: renamed from J?; footprint (none) -> SeeedOPL-Connector-2016:HW4-2.0
- J10, J11: renamed from J?; footprint (none) -> Connectors:1X01
- J2, J3, J4, J5: renamed from J?; footprint (none) -> capSensingStuff:SensePad
- JP1: renamed from JP?; footprint (none) -> Jumpers:SMT-JUMPER_2_NO_SILK
- R1, R10, R11, R12, R13, R14, R2, R3, R4, R5, R6, R7, R8, R9: renamed from R?; footprint (none) -> Resistors_SMD:R_0603_HandSoldering
- TH1: renamed from TH?; footprint (none) -> Resistors_SMD:R_0603_HandSoldering
- U1: renamed from U?; footprint (none) -> digikey-footprints:VOC_Sensor_LGA-10-1EP-2.7x4mm_CCS811B
- U2: renamed from U?; footprint (none) -> Housings_DFN_QFN:QFN-24_4x4mm_Pitch0.5mm_NoMask
Connections:
- net labels added: East, North, NorthEast, NorthWest, South, SouthEast, SouthWest, West
- wire segments 104 -> 192
- no-connect marks 3 -> 12
Other:
- note added: "CAP1188 - Cap Sensing Controller"
- note added: "CSS811 - VOC Sensor"
- note added: "I2C Connector"
- note added: "LED Interface"
- note added: "Power Flags"
- note added: "TCA9534 - IO Extender"

Commit message: up to revB
Parts:
- D11, D12, D13, D14, D15, D16, D17, D18: footprint LEDs:LED_0805_HandSoldering -> revLed:LED_1206_3216Metric_ReverseMount_Hole1.8x2.4mm
Changed lines of the file:
@@
 F 0 "D18" V 8646 2182 50  0000 R CNN
 F 1 "East" V 8555 2182 50  0000 R CNN
-F 2 "LEDs:LED_0805_HandSoldering" V 8600 2250 50  0001 C CNN
+F 2 "revLed:LED_1206_3216Metric_ReverseMount_Hole1.8x2.4mm" V 8600 2250 50  0001 C CNN
 F 3 "~" V 8600 2250 50  0001 C CNN
 	1    8600 2250
@@
 F 0 "D14" V 7525 1275 50  0000 R CNN
 F 1 "North" V 7425 1325 50  0000 R CNN
-F 2 "LEDs:LED_0805_HandSoldering" V 7500 1350 50  0001 C CNN
+F 2 "revLed:LED_1206_3216Metric_ReverseMount_Hole1.8x2.4mm" V 7500 1350 50  0001 C CNN
 F 3 "~" V 7500 1350 50  0001 C CNN
 	1    7500 1350
@@
 F 0 "D16" V 8146 1707 50  0000 R CNN
 F 1 "NorthEast" V 8055 1707 50  0000 R CNN
-F 2 "LEDs:LED_0805_HandSoldering" V 8100 1775 50  0001 C CNN
+F 2 "revLed:LED_1206_3216Metric_ReverseMount_Hole1.8x2.4mm" V 8100 1775 50  0001 C CNN
 F 3 "~" V 8100 1775 50  0001 C CNN
 	1    8100 1775
@@
 F 0 "D17" V 8146 2707 50  0000 R CNN
 F 1 "SouthEast" V 8055 2707 50  0000 R CNN
-F 2 "LEDs:LED_0805_HandSoldering" V 8100 2775 50  0001 C CNN
+F 2 "revLed:LED_1206_3216Metric_ReverseMount_Hole1.8x2.4mm" V 8100 2775 50  0001 C CNN
 F 3 "~" V 8100 2775 50  0001 C CNN
 	1    8100 2775
@@
 F 0 "D15" V 7546 3082 50  0000 R CNN
 F 1 "South" V 7455 3082 50  0000 R CNN
-F 2 "LEDs:LED_0805_HandSoldering" V 7500 3150 50  0001 C CNN
+F 2 "revLed:LED_1206_3216Metric_ReverseMount_Hole1.8x2.4mm" V 7500 3150 50  0001 C CNN
 F 3 "~" V 7500 3150 50  0001 C CNN
 	1    7500 3150
@@
 F 0 "D13" V 6996 2732 50  0000 R CNN
 F 1 "SouthWest" V 6875 2775 50  0000 R CNN
-F 2 "LEDs:LED_0805_HandSoldering" V 6950 2800 50  0001 C CNN
+F 2 "revLed:LED_1206_3216Metric_ReverseMount_Hole1.8x2.4mm" V 6950 2800 50  0001 C CNN
 F 3 "~" V 6950 2800 50  0001 C CNN
 	1    6950 2800
@@
 F 0 "D11" V 6471 2257 50  0000 R CNN
 F 1 "West" V 6380 2257 50  0000 R CNN
-F 2 "LEDs:LED_0805_HandSoldering" V 6425 2325 50  0001 C CNN
+F 2 "revLed:LED_1206_3216Metric_ReverseMount_Hole1.8x2.4mm" V 6425 2325 50  0001 C CNN
 F 3 "~" V 6425 2325 50  0001 C CNN
 	1    6425 2325
@@
 F 0 "D12" V 6996 1682 50  0000 R CNN
 F 1 "NorthWest" V 6875 1750 50  0000 R CNN
-F 2 "LEDs:LED_0805_HandSoldering" V 6950 1750 50  0001 C CNN
+F 2 "revLed:LED_1206_3216Metric_ReverseMount_Hole1.8x2.4mm" V 6950 1750 50  0001 C CNN
 F 3 "~" V 6950 1750 50  0001 C CNN
 	1    6950 1750

Commit message: REV C
Parts:
- removed D1, D2: 1N4148, Diodes_SMD:D_SOD-123, symbol Diode:1N4148
- removed J10, J11: Conn_01x01, Connectors:1X01, symbol Connector_Generic:Conn_01x01
- removed JP1: SolderJumper_2_Bridged, Jumpers:SMT-JUMPER_2_NO_SILK, symbol Jumper:SolderJumper_2_Bridged
- removed R9: 100K, Resistors_SMD:R_0603_HandSoldering, symbol Device:R_Small
- added R9: 10K, Resistors_SMD:R_0603_HandSoldering, symbol bikesenseCap-rescue:R_Small-Device
- D11, D12, D13, D14, D15, D16, D17, D18, D3, D4, D5, D6: symbol Device:LED_Small -> bikesenseCap-rescue:LED_Small-Device
- J1: symbol Connector:Conn_01x04_Male -> bikesenseCap-rescue:Conn_01x04_Male-Connector
- J2, J3, J4, J5: symbol cap1188:PAD -> bikesenseCap-rescue:PAD-cap1188
- R1, R10, R11, R12, R13, R14, R19, R2, R20, R21, R22, R23, R24, R25, R26, R27, R28, R29, R3, R30, R31, R32, R33, R34, R35, R36, R4, R5, R6, R7, R8: symbol Device:R_Small -> bikesenseCap-rescue:R_Small-Device
- TH1: symbol Device:Thermistor_NTC -> bikesenseCap-rescue:Thermistor_NTC-Device
- U1: symbol ccs811:CCS811 -> bikesenseCap-rescue:CCS811-ccs811
- U2: symbol cap1188:cap1188 -> bikesenseCap-rescue:cap1188-cap1188
- U3: symbol Interface_Expansion:TCA9534 -> bikesenseCap-rescue:TCA9534-Interface_Expansion
Connections:
- wire segments 192 -> 190

Commit message: REV C
Parts:
- J1: Arrow# (none) -> 110990037
- R19, R21, R22, R27, R28, R31, R32, R35: value 66 -> 100
Changed lines of the file:
@@
 F 1 "Conn_01x04_Male" H 1050 825 50  0000 C CNN
 F 2 "SeeedOPL-Connector-2016:HW4-2.0" H 1000 1100 50  0001 C CNN
-F 3 "~" H 1000 1100 50  0001 C CNN
+F 3 "https://www.arrow.com/en/products/110990037/seeed-technology-limited" H 1000 1100 50  0001 C CNN
+F 4 "110990037" H 1000 1100 50  0001 C CNN "Arrow#"
 	1    1000 1100
 	1    0    0    -1
@@
 P 8600 1950
 F 0 "R35" H 8659 1996 50  0000 L CNN
-F 1 "66" V 8600 1900 50  0000 L CNN
+F 1 "100" V 8600 1900 50  0000 L CNN
 F 2 "Resistors_SMD:R_0603_HandSoldering" H 8600 1950 50  0001 C CNN
 F 3 "~" H 8600 1950 50  0001 C CNN
@@
 P 7500 1050
 F 0 "R27" H 7350 1100 50  0000 L CNN
-F 1 "66" V 7500 1000 50  0000 L CNN
+F 1 "100" V 7500 1000 50  0000 L CNN
 F 2 "Resistors_SMD:R_0603_HandSoldering" H 7500 1050 50  0001 C CNN
 F 3 "~" H 7500 1050 50  0001 C CNN
@@
 P 8100 1475
 F 0 "R31" H 8159 1521 50  0000 L CNN
-F 1 "66" V 8100 1425 50  0000 L CNN
+F 1 "100" V 8100 1425 50  0000 L CNN
 F 2 "Resistors_SMD:R_0603_HandSoldering" H 8100 1475 50  0001 C CNN
 F 3 "~" H 8100 1475 50  0001 C CNN
@@
 P 8100 2475
 F 0 "R32" H 8159 2521 50  0000 L CNN
-F 1 "66" V 8100 2425 50  0000 L CNN
+F 1 "100" V 8100 2425 50  0000 L CNN
 F 2 "Resistors_SMD:R_0603_HandSoldering" H 8100 2475 50  0001 C CNN
 F 3 "~" H 8100 2475 50  0001 C CNN
@@
 P 7500 2850
 F 0 "R28" H 7559 2896 50  0000 L CNN
-F 1 "66" V 7500 2800 50  0000 L CNN
+F 1 "100" V 7500 2800 50  0000 L CNN
 F 2 "Resistors_SMD:R_0603_HandSoldering" H 7500 2850 50  0001 C CNN
 F 3 "~" H 7500 2850 50  0001 C CNN
@@
 P 6950 2500
 F 0 "R22" H 7009 2546 50  0000 L CNN
-F 1 "66" V 6950 2450 50  0000 L CNN
+F 1 "100" V 6950 2450 50  0000 L CNN
 F 2 "Resistors_SMD:R_0603_HandSoldering" H 6950 2500 50  0001 C CNN
 F 3 "~" H 6950 2500 50  0001 C CNN
@@
 P 6425 2025
 F 0 "R19" H 6484 2071 50  0000 L CNN
-F 1 "66" V 6425 1975 50  0000 L CNN
+F 1 "100" V 6425 1975 50  0000 L CNN
 F 2 "Resistors_SMD:R_0603_HandSoldering" H 6425 2025 50  0001 C CNN
 F 3 "~" H 6425 2025 50  0001 C CNN
@@
 P 6950 1450
 F 0 "R21" H 7009 1496 50  0000 L CNN
-F 1 "66" V 6950 1400 50  0000 L CNN
+F 1 "100" V 6950 1400 50  0000 L CNN
 F 2 "Resistors_SMD:R_0603_HandSoldering" H 6950 1450 50  0001 C CNN
 F 3 "~" H 6950 1450 50  0001 C CNN

Commit message: update
Parts:
- removed R10: 100K, Resistors_SMD:R_0603_HandSoldering, symbol bikesenseCap-rescue:R_Small-Device
- removed TH1: 10K ntc, Resistors_SMD:R_0603_HandSoldering, symbol bikesenseCap-rescue:Thermistor_NTC-Device
- removed U1: CCS811, digikey-footprints:VOC_Sensor_LGA-10-1EP-2.7x4mm_CCS811B, symbol bikesenseCap-rescue:CCS811-ccs811
- added AE1: W3011, antenna:w3011, symbol Device:Antenna_Shield
- added J6: ufl, .pretty:ufl, symbol ufl:ufl
- added U1: bme680, kicad-libraries:BME680, symbol bme680:bme680
- R7: value 100K -> 10K
Connections:
- net +3V3: now also R7.2, U1.6 (VDDIO), U1.8 (VDD); no longer R7.1
- net GND: now also U1.1 (GND), U1.7 (GND); no longer R7.2
- net SCL: now also U1.4 (SCL)
- net SDA: now also R7.1, U1.3 (SDA); no longer R8.1
- net at R9.1: now also U1.5 (SDO)
- new net: R8.1, U1.2 (CSB)
- new net: AE1.1 (A), J6.2 (SIG)
- new net GNDS: AE1.2 (Shield), J6.1 (GND)
- no-connect marks 12 -> 11
Other:
- note added: "BME680 - VOC Sensor"
- note added: "W3011 - Antenna"
- note removed: "CSS811 - VOC Sensor"

Commit message: Removed GPS and CAPsenseing led from broad
Parts:
- removed AE1: W3011, antenna:w3011, symbol Device:Antenna_Shield
- removed D3, D4, D5, D6: LED_Small, LEDs:LED_0603_HandSoldering, symbol bikesenseCap-rescue:LED_Small-Device
- removed J6: ufl, .pretty:ufl, symbol ufl:ufl
- removed R11, R12, R13, R14: 470, Resistors_SMD:R_0603_HandSoldering, symbol bikesenseCap-rescue:R_Small-Device
- U1: symbol bme680:bme680 -> bikesenseCap-rescue:bme680-bme680
Connections:
- no-connect marks 11 -> 15
Changed lines of the file:
@@
 EESchema Schematic File Version 4
 LIBS:bikesenseCap-cache
-EELAYER 26 0
+EELAYER 29 0
 EELAYER END
 $Descr User 9843 7874
@@
 Sheet 1 1
 Title "Bike Sense Daughter Board"
-Date "2019-05-10"
-Rev "PROD A"
+Date "2019-07-31"
+Rev "PROD B"
 Comp "David Dressner"
 Comment1 ""
@@
 Wire Wire Line
 	4000 1425 4150 1425
-$Comp
-L bikesenseCap-rescue:LED_Small-Device D6
-U 1 1 5BE39893
-P 4875 1725
-F 0 "D6" H 4975 1775 50  0000 C CNN
-F 1 "LED_Small" H 4875 1611 50  0001 C CNN
-F 2 "LEDs:LED_0603_HandSoldering" V 4875 1725 50  0001 C CNN
-F 3 "~" V 4875 1725 50  0001 C CNN
-	1    4875 1725
-	1    0    0    -1
-$EndComp
-$Comp
-L bikesenseCap-rescue:LED_Small-Device D5
-U 1 1 5BE398DF
-P 4875 1525
-F 0 "D5" H 4975 1575 50  0000 C CNN
-F 1 "LED_Small" H 4875 1411 50  0001 C CNN
-F 2 "LEDs:LED_0603_HandSoldering" V 4875 1525 50  0001 C CNN
-F 3 "~" V 4875 1525 50  0001 C CNN
-	1    4875 1525
-	1    0    0    -1
-$EndComp
-$Comp
-L bikesenseCap-rescue:LED_Small-Device D4
-U 1 1 5BE39929
-P 4875 1325
-F 0 "D4" H 4975 1375 50  0000 C CNN
-F 1 "LED_Small" H 4875 1211 50  0001 C CNN
-F 2 "LEDs:LED_0603_HandSoldering" V 4875 1325 50  0001 C CNN
-F 3 "~" V 4875 1325 50  0001 C CNN
-	1    4875 1325
-	1    0    0    -1
-$EndComp
-$Comp
-L bikesenseCap-rescue:LED_Small-Device D3
-U 1 1 5BE39981
-P 4875 1125
-F 0 "D3" H 4975 1175 50  0000 C CNN
-F 1 "LED_Small" H 4875 1011 50  0001 C CNN
-F 2 "LEDs:LED_0603_HandSoldering" V 4875 1125 50  0001 C CNN
-F 3 "~" V 4875 1125 50  0001 C CNN
-	1    4875 1125
-	1    0    0    -1
-$EndComp
-Wire Wire Line
-	4775 1125 4000 1125
-Wire Wire Line
-	4775 1325 4000 1325
-Wire Wire Line
-	4775 1525 4000 1525
-Wire Wire Line
-	4000 1725 4775 1725
-$Comp
-L bikesenseCap-rescue:R_Small-Device R11
-U 1 1 5BE3C213
-P 5225 1125
-F 0 "R11" V 5300 1050 50  0000 R CNN
-F 1 "470" V 5225 1200 50  0000 R CNN
-F 2 "Resistors_SMD:R_0603_HandSoldering" H 5225 1125 50  0001 C CNN
-F 3 "~" H 5225 1125 50  0001 C CNN
-	1    5225 1125
-	0    -1   -1   0
-$EndComp
-$Comp
-L bikesenseCap-rescue:R_Small-Device R12
-U 1 1 5BE3C437
-P 5225 1325
-F 0 "R12" V 5300 1250 50  0000 R CNN
-F 1 "470" V 5225 1400 50  0000 R CNN
-F 2 "Resistors_SMD:R_0603_HandSoldering" H 5225 1325 50  0001 C CNN
-F 3 "~" H 5225 1325 50  0001 C CNN
-	1    5225 1325
-	0    -1   -1   0
-$EndComp
-$Comp
-L bikesenseCap-rescue:R_Small-Device R13
-U 1 1 5BE3C48B
-P 5225 1525
-F 0 "R13" V 5300 1450 50  0000 R CNN
-F 1 "470" V 5225 1600 50  0000 R CNN
-F 2 "Resistors_SMD:R_0603_HandSoldering" H 5225 1525 50  0001 C CNN
-F 3 "~" H 5225 1525 50  0001 C CNN
-	1    5225 1525
-	0    -1   -1   0
-$EndComp
-$Comp
-L bikesenseCap-rescue:R_Small-Device R14
-U 1 1 5BE3C4DD
-P 5225 1725
-F 0 "R14" V 5300 1650 50  0000 R CNN
-F 1 "470" V 5225 1800 50  0000 R CNN
-F 2 "Resistors_SMD:R_0603_HandSoldering" H 5225 1725 50  0001 C CNN
-F 3 "~" H 5225 1725 50  0001 C CNN
-	1    5225 1725
-	0    -1   -1   0
-$EndComp
-Wire Wire Line
-	5125 1125 4975 1125
-Wire Wire Line
-	4975 1325 5125 1325
-Wire Wire Line
-	5125 1525 4975 1525
-Wire Wire Line
-	4975 1725 5125 1725
-$Comp
-L bikesenseCap-rescue:+3V3-power #PWR0107
-U 1 1 5BE414C9
-P 5550 1050
-F 0 "#PWR0107" H 5550 900 50  0001 C CNN
-F 1 "+3V3" H 5565 1223 50  0000 C CNN
-F 2 "" H 5550 1050 50  0001 C CNN
-F 3 "" H 5550 1050 50  0001 C CNN
-	1    5550 1050
-	1    0    0    -1
-$EndComp
-Wire Wire Line
-	5550 1050 5550 1125
-Wire Wire Line
-	5550 1125 5325 1125
-Wire Wire Line
-	5325 1325 5550 1325
-Wire Wire Line
-	5550 1325 5550 1125
-Connection ~ 5550 1125
-Wire Wire Line
-	5325 1525 5550 1525
-Wire Wire Line
-	5550 1525 5550 1325
-Connection ~ 5550 1325
-Wire Wire Line
-	5325 1725 5550 1725
-Wire Wire Line
-	5550 1725 5550 1525
-Connection ~ 5550 1525
 $Comp
 L bikesenseCap-rescue:TCA9534-Interface_Expansion U3
@@
 NoConn ~ 4000 2625
 $Comp
-L bme680:bme680 U1
+L bikesenseCap-rescue:bme680-bme680 U1
 U 1 1 5C81009D
 P 1600 4850
@@
 W3011 - Antenna
 $Comp
-L Device:Antenna_Shield AE1
-U 1 1 5CD75914
-P 4450 3950
-F 0 "AE1" H 4590 3991 50  0000 L CNN
-F 1 "W3011" H 4590 3900 50  0000 L CNN
-F 2 "antenna:w3011" H 4450 4050 50  0001 C CNN
-F 3 "~" H 4450 4050 50  0001 C CNN
-	1    4450 3950
-	1    0    0    -1
-$EndComp
-$Comp
-L ufl:ufl J6
-U 1 1 5CD75B95
-P 4025 4725
-F 0 "J6" H 4025 5140 50  0000 C CNN
-F 1 "ufl" H 4025 5049 50  0000 C CNN
-F 2 ".pretty:ufl" H 4025 4725 50  0001 C CNN
-F 3 "" H 4025 4725 50  0001 C CNN
-	1    4025 4725
-	1    0    0    -1
-$EndComp
-Wire Wire Line
-	4450 4150 4450 4725
-Wire Wire Line
-	4450 4725 4225 4725
-$Comp
-L power:GNDS #PWR0108
-U 1 1 5CD7E2DA
-P 4550 4275
-F 0 "#PWR0108" H 4550 4025 50  0001 C CNN
-F 1 "GNDS" H 4555 4102 50  0000 C CNN
-F 2 "" H 4550 4275 50  0001 C CNN
-F 3 "" H 4550 4275 50  0001 C CNN
-	1    4550 4275
-	1    0    0    -1
-$EndComp
-Wire Wire Line
-	4550 4150 4550 4275
-$Comp
-L power:GNDS #PWR0109
-U 1 1 5CD86B4A
-P 4025 5200
-F 0 "#PWR0109" H 4025 4950 50  0001 C CNN
-F 1 "GNDS" H 4030 5027 50  0000 C CNN
-F 2 "" H 4025 5200 50  0001 C CNN
-F 3 "" H 4025 5200 50  0001 C CNN
-	1    4025 5200
-	1    0    0    -1
-$EndComp
-Wire Wire Line
-	4025 5200 4025 5075
-$Comp
 L bikesenseCap-rescue:Conn_01x04_Male-Connector J1
 U 1 1 5BE338ED
@@
 	1    0    0    -1
 $EndComp
+NoConn ~ 4000 1125
+NoConn ~ 4000 1325
+NoConn ~ 4000 1525
+NoConn ~ 4000 1725
 $EndSCHEMATC
